Commit message: fix urdf

File: forklift_robot_description/urdf/forklift_robot.urdf (robot description, URDF)
Before this commit: robot forklift_robot, 6 links, 5 joints
Links:
- link wheel_back_left: geometry collision mesh filename=package://forklift_robot_description/meshes/wheel.dae; visual mesh filename=package://forklift_robot_description/meshes/wheel.dae
- link wheel_back_right: geometry collision mesh filename=package://forklift_robot_description/meshes/wheel.dae; visual mesh filename=package://forklift_robot_description/meshes/wheel.dae
- link wheel_front_left: geometry collision mesh filename=package://forklift_robot_description/meshes/wheel.dae; visual mesh filename=package://forklift_robot_description/meshes/wheel.dae
- link wheel_front_right: geometry collision mesh filename=package://forklift_robot_description/meshes/wheel.dae; visual mesh filename=package://forklift_robot_description/meshes/wheel.dae
Joints:
- joint base_to_fork: origin xyz=1.0795 -0.3686 0.0 -> (none)
- joint base_to_wheel_back_left: origin xyz=-0.7865 -0.5334 0.2032 -> (none); type continuous -> revolute
- joint base_to_wheel_back_right: origin xyz=-0.7502 0.3302 0.2032 -> (none); type continuous -> revolute
- joint base_to_wheel_front_left: origin xyz=0.6722 0.3302 0.2032 -> (none); type continuous -> revolute
- joint base_to_wheel_front_right: origin xyz=0.6722 -0.5334 0.2032 -> (none); type continuous -> revolute

Commit message: back to original urdf: link has no pose

File: forklift_robot_description/urdf/forklift_robot.urdf (robot description, URDF)
Before this commit: robot forklift_robot, 6 links, 5 joints
Links:
- link wheel_back_left: geometry collision cylinder length=0.2 radius=0.21; visual mesh filename=package://forklift_robot_description/meshes/wheel.dae
- link wheel_back_right: geometry collision cylinder length=0.2 radius=0.21; visual mesh filename=package://forklift_robot_description/meshes/wheel.dae
- link wheel_front_left: geometry collision cylinder length=0.2 radius=0.21; visual mesh filename=package://forklift_robot_description/meshes/wheel.dae
- link wheel_front_right: geometry collision cylinder length=0.2 radius=0.21; visual mesh filename=package://forklift_robot_description/meshes/wheel.dae
Joints:
- joint base_to_fork: origin (none) -> xyz=1.0795 -0.3686 0.0
- joint base_to_wheel_back_left: origin (none) -> xyz=-0.7865 -0.5334 0.2032; type revolute -> continuous
- joint base_to_wheel_back_right: origin (none) -> xyz=-0.7502 0.3302 0.2032; type revolute -> continuous
- joint base_to_wheel_front_left: origin (none) -> xyz=0.6722 0.3302 0.2032; type revolute -> continuous
- joint base_to_wheel_front_right: origin (none) -> xyz=0.6722 -0.5334 0.2032; type revolute -> continuous
